Commit message: Add files via upload

File: drone_description.urdf (robot description, URDF)
Before this commit: robot drone, 7 links, 6 joints
Links:
- added link gimbal_camera_optical_frame
- added link landing_center_point; visual sphere radius=0.01
Joints:
- added joint gimbal_camera_optical_joint: type fixed, parent gimbal_camera_link, child gimbal_camera_optical_frame, origin xyz=0 0 0 rpy=-1.57079632679 0 -1.57079632679
- added joint landing_center_joint: type fixed, parent base_link, child landing_center_point, origin xyz=0.02 0 -0.055 rpy=0 0 0
